File: theremin.kicad_pcb (KiCad board)
At the start: 2 copper layers, 64 parts, among them IC1 LM386, P1 PITCH ANT, P2 VOLUME ANT, Q1 2N2222, Q2 2N2222, Q3 PN3640, Q4 2N2222, Q5 PN3640, Q6 2N2222, Q7 PN3640, Q8 PN5089, Q9 2N2222

Commit message: Corrected some footprints in PCB.
Parts:
- C8: footprint Capacitors_ThroughHole:Capacitor5x11RM2.5 -> Capacitors_ThroughHole:Capacitor4x3RM2.5
- moved L3 197.6 mm to (245.1, 128.3), turned to 90 degrees
- moved R21 191.8 mm to (215.9, 129.5), turned to 180 degrees
- moved Q5 167.9 mm to (236.2, 149.9)
- moved C5 160.9 mm to (153.7, 149.9), turned to 270 degrees
- moved R7 152.7 mm to (134.6, 153.7), turned to 270 degrees
- moved L2 147.6 mm to (146.1, 147.3), turned to 270 degrees
- moved P2 136.7 mm to (160.0, 146.1), turned to 270 degrees
- moved C6 126.7 mm to (138.4, 135.9), turned to 270 degrees
- moved C7 124.8 mm to (132.1, 143.5), turned to 180 degrees
- moved R8 122.6 mm to (125.7, 121.9)
- moved L4 116.3 mm to (43.2, 146.1), turned to 270 degrees
- moved R17 115.9 mm to (138.4, 80.0), turned to 90 degrees
- moved R20 115.6 mm to (139.7, 123.2), turned to 90 degrees
- moved R23 114.5 mm to (132.1, 110.5), turned to 180 degrees
- moved C15 111.9 mm to (146.1, 73.7), turned to 180 degrees
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Routing:
- net Net-(C19-Pad2): track 5.08 -> 0.00 mm
